File: pcb/fan-control.kicad_sch (KiCad schematic)
At the start: 23 parts, among them J1 USB_C_Receptacle_USB2.0_14P, J2 USB_C_Receptacle_USB2.0_14P, Q1 BSS138, SW1 SW_Push, U1 ESP32-C6-WROOM-1-N8

Commit message: schematic
Parts:
- added C2: 10u, symbol Device:C
- added C3: 22u, symbol Device:C
- added R10, R11, R12, R13, R14, R15, R16, R17, R8, R9: 1k, symbol Device:R
- added R18: 100k, symbol Device:R
- added R19, R20: R, symbol Device:R
- added U2: MPM3610GQV-P, MPM3610GQV-P:CONV_MPM3610GQV-P, symbol MPM3610GQV-P:MPM3610GQV-P
Connections:
- net +10V: now also C2.1, R18.1, U2.16 (IN)
- net +3V3: now also C3.1, R10.1, R11.1, R12.1, R13.1, R14.1, R15.1, R16.1, R17.1, R19.1, R8.1, R9.1, U2.7 (OUT)
- net GND: now also C2.2, C3.2, R20.2, U2.12 (PGND), U2.13 (PGND), U2.14 (PGND), U2.3 (AGND)
- net LED1: now reaches D1.1 (K)
- net LED1: now also U1.12 (IO11)
- net at D1.2 (A): now also R8.2
- net LED10: now reaches D10.1 (K)
- net LED10: now also U1.21 (IO23)
- net at D10.2 (A): now also R17.2
- net LED3: now reaches D3.1 (K)
- net LED3: now also U1.25 (TXD0/GPIO16)
- net at D3.2 (A): now also R10.2
- net LED7: now reaches D7.1 (K)
- net LED7: now also U1.18 (IO20)
- net at D7.2 (A): now also R14.2
- net LED8: now reaches D8.1 (K)
- net LED8: now also U1.19 (IO21)
- net at D8.2 (A): now also R15.2
- net LED5: now reaches U1.16 (IO18)
- net LED5: now also D5.1 (K)
- net LED6: now reaches U1.17 (IO19)
- net LED6: now also D6.1 (K)
- net LED9: now reaches U1.20 (IO22)
- net LED9: now also D9.1 (K)
- net LED2: now reaches U1.23 (IO15)
- net LED2: now also D2.1 (K)
- net LED4: now reaches U1.24 (RXD0/GPIO17)
- net LED4: now also D4.1 (K)
- net at D5.2 (A): now also R12.2
- net at D4.2 (A): now also R11.2
- net at D9.2 (A): now also R16.2
- net at D6.2 (A): now also R13.2
- net at D2.2 (A): now also R9.2
- new net: R18.2, U2.17 (EN)
- new net: R19.2, R20.1
Other:
- moved on the sheet: C1, D1, D10, D2, D3, D4, D5, D6, D7, D8, D9, Q1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

Commit message: More sch
Parts:
- added C4: 0.1u, symbol Device:C
- added R21: 10k, symbol Device:R
- added SW2: SW_Push, symbol Switch:SW_Push
- R18: value 100k -> 75k
- R19: value R -> 75k
- R20: value R -> 24k
Connections:
- net +10V: now also R18.2; no longer R18.1
- net +3V3: now also R21.1
- net BOOT: now also C4.1, R21.2, SW2.2
- net GND: now also C4.2, SW2.1
- net at U2.17 (EN): now also R18.1; no longer R18.2
- net BUTTON: now reaches U1.8 (IO0)
- net BUTTON: now also C1.1, R7.2, SW1.2
- net at R19.2, R20.1: now also U2.1 (FB)
- net PWM_OUT renamed ESP_PWM
Other:
- note added: "Boot Button"
- note added: "SMPS 10V -> 3V3"
- title: (none) -> UIS Fan Controller
- moved on the sheet: C1, C2, C3, D1, D10, D2, D3, D4, D5, D6, D7, D8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

Commit message: Outline
Parts:
- added H1, H2, H3: MountingHole, MountingHole:MountingHole_2.2mm_M2, symbol Mechanical:MountingHole
- added R22, R23: 47k, Resistor_SMD:R_0603_1608Metric_Pad0.98x0.95mm_HandSolder, symbol Device:R
- C1, C4: footprint (none) -> Capacitor_SMD:C_0603_1608Metric_Pad1.08x0.95mm_HandSolder
- C2, C3: footprint (none) -> Capacitor_SMD:C_0805_2012Metric_Pad1.18x1.45mm_HandSolder
- D1, D10, D2, D3, D4, D5, D6, D7, D8, D9: footprint (none) -> LED_SMD:LED_0603_1608Metric_Pad1.05x0.95mm_HandSolder
- J1, J2: footprint (none) -> Connector_USB:USB_C_Receptacle_GCT_USB4105-xx-A_16P_TopMnt_Horizontal
- R1, R10, R11, R12, R13, R14, R15, R16, R17, R18, R19, R2, R20, R21, R3, R4, R5, R6, R7, R8, R9: footprint (none) -> Resistor_SMD:R_0603_1608Metric_Pad0.98x0.95mm_HandSolder
- SW1, SW2: footprint (none) -> Button_Switch_THT:SW_PUSH_6mm
- U1: footprint ESP32-C6-WROOM-1-N8:XCVR_ESP32-C6-WROOM-1-N8 -> SnapEDA:XCVR_ESP32-C6-WROOM-1-N8
- U2: footprint MPM3610GQV-P:CONV_MPM3610GQV-P -> SnapEDA:CONV_MPM3610GQV-P
Connections:
- net +10V: now also J1.A4 (VBUS), J1.A9 (VBUS), J1.B4 (VBUS), J1.B9 (VBUS), R22.1
- net FAN_PWM: now also J1.A6 (D+), J1.B6 (D+)
- net GND: now also R23.2
- net at J1.A5 (CC1): now also R22.2, R23.1
- net TACH: now reaches J1.A7 (D-)
- net TACH: now also J1.B7 (D-)
Other:
- moved on the sheet: J1

Commit message: some layout
Parts:
- SW1, SW2: footprint Button_Switch_THT:SW_PUSH_6mm -> Footprints:4P-3.4x3.4mm
Connections:
- net +3V3: now also D1.2 (A), D10.2 (A), D2.2 (A), D3.2 (A), D4.2 (A), D5.2 (A), D6.2 (A), D7.2 (A), D8.2 (A), D9.2 (A); no longer R10.1, R11.1, R12.1, R13.1, R14.1, R15.1, R16.1, R17.1, R8.1, R9.1
- net LED1: now also R8.2; no longer D1.1 (K)
- net LED10: now also R17.2; no longer D10.1 (K)
- net LED2: now also R9.2; no longer D2.1 (K)
- net LED3: now also R10.2; no longer D3.1 (K)
- net LED4: now also R11.2; no longer D4.1 (K)
- net LED5: now also R12.2; no longer D5.1 (K)
- net LED6: now also R13.2; no longer D6.1 (K)
- net LED7: now also R14.2; no longer D7.1 (K)
- net LED8: now also R15.2; no longer D8.1 (K)
- net LED9: now also R16.2; no longer D9.1 (K)
- new net: D1.1 (K), R8.1
- new net: D9.1 (K), R16.1
- new net: D10.1 (K), R17.1
- new net: D6.1 (K), R13.1
- new net: D2.1 (K), R9.1
- new net: D3.1 (K), R10.1
- new net: D7.1 (K), R14.1
- new net: D8.1 (K), R15.1
- new net: D5.1 (K), R12.1
- new net: D4.1 (K), R11.1
Other:
- moved on the sheet: D1, D10, D2, D3, D4, D5, D6, D7, D8, D9, R10, R11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

Commit message: Routing
Parts:
- removed J2: USB_C_Receptacle_USB2.0_14P, Connector_USB:USB_C_Receptacle_GCT_USB4105-xx-A_16P_TopMnt_Horizontal, symbol Connector:USB_C_Receptacle_USB2.0_14P
- removed R3, R4: 5.1k, Resistor_SMD:R_0603_1608Metric_Pad0.98x0.95mm_HandSolder, symbol Device:R
- added J3: Conn_ARM_SWD_TagConnect_TC2030-NL, Connector:Tag-Connect_TC2030-IDC-NL_2x03_P1.27mm_Vertical, symbol Connector:Conn_ARM_SWD_TagConnect_TC2030-NL
Connections:
- net D+ is gone; now on net LED4: U1.14 (IO13)
- net +3V3: now also J3.1 (VCC)
- net ESP_PWM: now also U1.5 (IO5)
- net GND: now also J3.5 (GND)
- net LED1: now also R11.2, U1.26 (IO3); no longer R8.2, U1.12 (IO11)
- net LED10: now also R10.2; no longer R17.2
- net LED2: now also R13.2; no longer R9.2
- net LED3: now also R12.2, U1.27 (IO2); no longer R10.2, U1.25 (TXD0/GPIO16)
- net LED4: now also R16.2; no longer R11.2, U1.24 (RXD0/GPIO17)
- net LED5: now also R15.2; no longer R12.2
- net LED6: now also R17.2; no longer R13.2
- net LED7: now also R8.2; no longer R14.2
- net LED8: now also R14.2; no longer R15.2
- net LED9: now also R9.2; no longer R16.2
- net D-: no longer names the net of U1.13 (IO12)
- new net RX: J3.2 (SWDIO), U1.24 (RXD0/GPIO17)
- new net TX: J3.4 (SWCLK), U1.25 (TXD0/GPIO16)
Other:
- note added: "Mechanical Support"
- moved on the sheet: C1, C4, H1, H2, H3, R2, R21, R7, SW1, SW2

Commit message: drc, nearing end of layout
Parts:
- added TP1: TestPoint, TestPoint:TestPoint_Pad_1.5x1.5mm, symbol Connector:TestPoint
Connections:
- net TACH: now also TP1.1
- no-connect marks 0 -> 4
Other:
- moved on the sheet: J1, R22, R23

Commit message: Add switch comment
Other:
- note added: "TODO: Button footprint doesn't match reality"
- note added: "TODO: Mounting holes off a bit"
Changed lines of the file:
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@@
+		)
+	)
+	(text "TODO: Button footprint doesn't match reality\n"
+		(exclude_from_sim no)
+		(at 126.492 133.35 0)
+		(effects
+			(font
+				(size 1.27 1.27)
+				(color 255 0 255 1)
+			)
 		)
 	)
@@
 			)
 		)
+	)
+	(text "TODO: Mounting holes off a bit"
+		(exclude_from_sim no)
+		(at 195.834 168.402 0)
+		(effects
+			(font
+				(size 1.27 1.27)
+				(color 255 0 255 1)
+			)
+		)
